Commit message: 可以初步探索，但uav1不动，剩下3架无人机也只是探索一小部分区域

File: src/RACER/swarm_exploration/rotors_simulator/rotors_gazebo/models/rotors_description/urdf/component_snippets.xacro (robot description, xacro)
@@ -304,4 +304,5 @@
         <odometryTopic>${odometry_topic}</odometryTopic>
         <parentFrameId>${parent_frame_id}</parentFrameId>  <!-- Use the scoped link name here. e.g. Model::link. -->
+        <childFrameId>${namespace}/odometry_sensor${odometry_sensor_suffix}_link</childFrameId>
         <measurementDivisor>${measurement_divisor}</measurementDivisor> <!-- only every (seq % measurementDivisor) == 0 measurement is published [int] -->
         <measurementDelay>${measurement_delay}</measurementDelay> <!-- time that measurement gets held back before it's published in [simulation cycles (int)] -->
@@ -389,5 +390,5 @@
     <link name="${namespace}/camera_${camera_suffix}_optical_center_link" />
     <joint name="${namespace}/camera_${camera_suffix}_optical_center_joint" type="fixed">
-      <origin xyz="0 0 0" rpy="${-PI/2} 0 ${-PI/2}" />
+      <origin xyz="0 0 0" rpy="-1.57079632679 0 -1.57079632679" />
       <parent link="${namespace}/camera_${camera_suffix}_link" />
       <child link="${namespace}/camera_${camera_suffix}_optical_center_link" />
@@ -415,5 +416,5 @@
           <baseline>0.11</baseline>
           <updateRate>${frame_rate}</updateRate>
-          <cameraName>camera_${camera_suffix}</cameraName>
+          <cameraName></cameraName>
           <imageTopicName>camera/image_raw</imageTopicName>
           <cameraInfoTopicName>camera/camera_info</cameraInfoTopicName>

File: src/RACER/swarm_exploration/rotors_simulator/rotors_gazebo/models/rotors_description/urdf/iris_base.xacro (robot description, xacro)
@@ -12,5 +12,5 @@
   <xacro:include filename="$(arg rotors_description_dir)/urdf/iris.xacro" />
   <!-- Bridge controller output to the Gazebo motor model command topic. -->
-  <xacro:controller_plugin_macro namespace="${namespace}" imu_sub_topic="imu" />
+  <xacro:controller_plugin_macro namespace="${namespace}" imu_sub_topic="imu/data" />
   <xacro:if value="$(arg enable_wind)">
     <xacro:wind_plugin_macro
@@ -29,5 +29,5 @@
   <xacro:mavlink_interface_macro
     namespace="${namespace}"
-    imu_sub_topic="/imu"
+    imu_sub_topic="imu/data"
     mavlink_addr="INADDR_ANY"
     mavlink_udp_port="14560"
@@ -40,5 +40,5 @@
     imu_suffix=""
     parent_link="base_link"
-    imu_topic="/imu"
+    imu_topic="imu/data"
     mass_imu_sensor="0.015"
     gyroscope_noise_density="0.0003394"
@@ -54,4 +54,12 @@
     <origin xyz="0 0 0" rpy="0 0 0" />
   </xacro:imu_plugin_macro>
+  <!-- Forward-facing depth camera for Gazebo/Racer map updates. -->
+  <xacro:vi_sensor_depth_macro
+    namespace="${namespace}"
+    parent_link="base_link"
+    camera_suffix="depth"
+    frame_rate="30.0">
+    <origin xyz="0.13 0 0.03" rpy="0 0 0" />
+  </xacro:vi_sensor_depth_macro>
   <xacro:if value="$(arg enable_ground_truth)">
     <!-- Mount an IMU providing ground truth. -->
