Commit message: 05.02修改后初步能飞

File: src/RACER/swarm_exploration/rotors_simulator/rotors_description/urdf/VLP-16.urdf.xacro (robot description, xacro)
@@ -89,5 +89,5 @@
             <!-- <robotNamespace>${namespace}</robotNamespace> -->
             <topicName>${topic}</topicName>
-            <frameName>${name}</frameName>
+            <frameName>${namespace}/${name}</frameName>
             <organize_cloud>${organize_cloud}</organize_cloud>
             <min_range>${min_range}</min_range>
@@ -131,5 +131,5 @@
             <!-- <robotNamespace>${namespace}</robotNamespace> -->
             <topicName>${topic}</topicName>
-            <frameName>${name}</frameName>
+            <frameName>${namespace}/${name}</frameName>
             <organize_cloud>${organize_cloud}</organize_cloud>
             <min_range>${min_range}</min_range>

File: src/RACER/swarm_exploration/rotors_simulator/rotors_description/urdf/ardrone.xacro (robot description, xacro)
@@ -17,5 +17,5 @@
   <xacro:property name="time_constant_up" value="0.0125" /> <!-- [s] -->
   <xacro:property name="time_constant_down" value="0.025" /> <!-- [s] -->
-  <xacro:property name="max_rot_velocity" value="838" /> <!-- [rad/s] -->
+  <xacro:property name="max_rot_velocity" value="1500" /> <!-- [rad/s] -->
   <xacro:property name="sin30" value="0.5" />
   <xacro:property name="cos30" value="0.866025403784" />
@@ -67,5 +67,5 @@
   <xacro:include filename="$(find rotors_description)/urdf/VLP-16.urdf.xacro" />
   <xacro:VLP-16 namespace="${namespace}" parent="${namespace}/base_lidar_support"  name="velodyne"
-    topic="/velodyne_points" hz="30" samples="300" min_range="0.1" organize_cloud="true" gpu="true"
+    topic="/${namespace}/velodyne_points" hz="30" samples="300" min_range="0.1" organize_cloud="true" gpu="true"
     support_height="${lidar_support_height}">
     <origin xyz="0 0 0" rpy="0 0 0" />
